File: PCB/LoadBoard/LoadBoard.kicad_pcb (KiCad board)
At the start: 2 copper layers, 115 x 126 mm, 7 parts

Commit message: Layout of load pcb
Parts:
- added H1: MountingHole, MountingHole:MountingHole_3.2mm_M3, F.Cu at (133.0, 141.0)
- added H2: MountingHole, MountingHole:MountingHole_3.2mm_M3, F.Cu at (238.0, 141.0)
- added H3: MountingHole, MountingHole:MountingHole_3.2mm_M3, F.Cu at (133.0, 25.0)
- added H4: MountingHole, MountingHole:MountingHole_3.2mm_M3, F.Cu at (238.0, 25.0)
- added J1: Conn_01x04, TerminalBlock_Phoenix:TerminalBlock_Phoenix_MKDS-1-4-3.81_1x04_P3.81mm_Horizontal, F.Cu at (135.0, 118.6)
- moved R5 15.0 mm to (154.0, 136.0)
- moved L3 8.49 mm to (159.0, 99.0)
- moved L2 3.61 mm to (155.0, 48.0), turned to 180 degrees
Connections:
- net Net-(J1-Pin_2) renamed /ramp_1
- net Net-(J1-Pin_3) renamed /main_h
- net Net-(J1-Pin_4) renamed /main_l
- L2 pad 1: Net-(J1-Pin_1) -> /ramp_2
Routing:
- net /main_h: track 0.00 -> 218.6 mm
- net /main_l: track 0.00 -> 150.1 mm
- net /ramp_1: track 0.00 -> 128.2 mm
- net /ramp_2: track 0.00 -> 72.0 mm
- added copper zone on B.Cu, net (none)
- added copper zone on F.Cu, net (none)
- added copper zone on B.Cu, net /main_h
- added copper zone on F.Cu, net /main_l
- added copper zone on B.Cu, net /ramp_1
- added copper zone on B.Cu, net /ramp_2
Other:
- outline, holes or cut-outs redrawn
- board text added: "12"
- board text added: "68"
- board text added: "7.5"
- board text added: "GND"
- board text added: "Reactive"
- board text added: "Resistive"
