File: PCB/LoadBoard/LoadBoard.kicad_sch (KiCad schematic)
At the start: 8 parts, among them J1 Conn_01x04

Commit message: Layout of load pcb
Parts:
- added H1, H2, H3, H4: MountingHole, MountingHole:MountingHole_3.2mm_M3, symbol Mechanical:MountingHole
- J1: footprint (none) -> TerminalBlock_Phoenix:TerminalBlock_Phoenix_MKDS-1-4-3.81_1x04_P3.81mm_Horizontal
Connections:
- net ramp_2: now reaches J1.1 (Pin_1), L2.1
- net ramp_1: now reaches J1.2 (Pin_2), L2.2, L3.1, R5.1
- net main_h: now reaches C1.1, C2.1, C3.1, J1.3 (Pin_3), L1.1, L3.2, R5.2
- net main_l: now reaches C1.2, C2.2, C3.2, J1.4 (Pin_4), L1.2
